File: Digital_Cape_2.0.kicad_pcb (KiCad board)
At the start: 2 copper layers, 54.6 x 86.4 mm, 30 parts, among them J1 RJ45, J2 RJ45, P8 BeagleBone_Black_Header, P9 BeagleBone_Black_Header, U1 CAT24C256, U2 BME_280, U3 LSM9_DS1

Commit message: Reposition RJ12 ports
Parts:
- moved J1 3.89 mm to (146.2, 120.0)
- moved J2 3.32 mm to (128.8, 120.0)
Routing:
- net /I2C2_SDA: track 99.9 -> 90.7 mm
- net /I2C2_SCL: track 91.9 -> 84.5 mm
- net /I2C1_SDA: track 96.3 -> 91.5 mm
- net /I2C1_SCL: track 89.8 -> 85.4 mm
- net +5V: track 92.5 -> 91.0 mm
